Commit message: Add example of a continuous relation

File: models/busybox/model.urdf (robot description, URDF)
Before this commit: robot busybox, 5 links, 4 joints
Links:
- added link door_handle, mass 0.25; collision box size=0.025 0.1 0.025; visual box size=0.025 0.1 0.025
- added link door_latch, mass 0.25; collision box size=0.05 0.05 0.05; visual box size=0.05 0.05 0.05
Joints:
- added joint prismatic_door_latch: type prismatic, parent base_link, child door_latch, origin xyz=0.2 -0.1 0.075 rpy=0 0 0, axis 0 1 0, limit lower=-0.1 upper=0
- added joint revolute_door_handle: type revolute, parent base_link, child door_handle, origin xyz=0 -0.1 0.0625 rpy=0 0 0, axis 0 0 1, limit lower=0 upper=1.0
