Commit message: changed spinner handle and spinner base to continuous revolute joints so easier to control

File: models/simple_busybox/model.urdf (robot description, URDF)
Before this commit: robot busybox, 4 links, 3 joints
Joints:
- removed joint fixed_spinner_handle
- added joint spinner_handle: type continuous, parent spinner, child spinner_handle, origin xyz=-0.075 0 0.075 rpy=0 0 0, axis 0 0 1, limit effort=100 velocity=100
- joint revolute_spinner: limit lower=-2.0 upper=2.0 effort=10 velocity=10 -> effort=10 velocity=10; type revolute -> continuous

Commit message: chaning name to slider

File: models/simple_busybox/model.urdf (robot description, URDF)
Before this commit: robot busybox, 4 links, 3 joints
Joints:
- removed joint prismatic_slider
- added joint slider: type prismatic, parent base_link, child slider, origin xyz=-0.2 0.0 0.075 rpy=0 0 0, axis 0 1 0, limit lower=-0.2 upper=0.2
