Commit message: Modified replay training algorithm

File: models/busybox0.urdf (robot description, URDF)
Before this commit: robot busybox, 4 links, 3 joints
Links:
- removed link slider_9_handle
- removed link slider_9_track
- added link slider_6_handle, mass 0.1; collision cylinder length=0.05 radius=0.02; visual cylinder length=0.05 radius=0.02
- added link slider_6_track, mass 0.1; collision box size=0.24386959843256184 0.005 0.02; visual box size=0.24386959843256184 0.005 0.02
Joints:
- removed joint slider_9_joint
- removed joint slider_9_track_joint
- added joint slider_6_joint: type prismatic, parent back_link, child slider_6_handle, origin xyz=0.03487218109430357 0.05 0.21680858279097454 rpy=1.57 0 0, axis -0.9820927964374071 0.18839782160564802 0, limit lower=-0.12193479921628092 upper=0.12193479921628092 effort=UNNAMED_12 velocity=UNNAMED_13
- added joint slider_6_track_joint: type fixed, parent back_link, child slider_6_track, origin xyz=0.03487218109430357 0.025 0.21680858279097454 rpy=0 -2.9520621552029778 0

Commit message: Modified validation error calc

File: models/busybox0.urdf (robot description, URDF)
Before this commit: robot busybox, 4 links, 3 joints
Links:
- removed link slider_6_handle
- removed link slider_6_track
- added link slider_72_handle, mass 0.1; collision cylinder length=0.05 radius=0.02; visual cylinder length=0.05 radius=0.02
- added link slider_72_track, mass 0.1; collision box size=0.3203024813295854 0.005 0.02; visual box size=0.3203024813295854 0.005 0.02
Joints:
- removed joint slider_6_joint
- removed joint slider_6_track_joint
- added joint slider_72_joint: type prismatic, parent back_link, child slider_72_handle, origin xyz=0.0396377531083687 0.05 0.0327181465653521 rpy=1.57 0 0, axis -0.7010127802428574 0.7131487095523481 0, limit lower=-0.1601512406647927 upper=0.1601512406647927 effort=UNNAMED_78 velocity=UNNAMED_79
- added joint slider_72_track_joint: type fixed, parent back_link, child slider_72_track, origin xyz=0.0396377531083687 0.025 0.0327181465653521 rpy=0 -2.3476129869551983 0

Commit message: Removed args.type

File: models/busybox0.urdf (robot description, URDF)
Before this commit: robot busybox, 4 links, 3 joints
Links:
- removed link slider_72_handle
- removed link slider_72_track
- added link slider_11_handle, mass 0.1; collision cylinder length=0.05 radius=0.02; visual cylinder length=0.05 radius=0.02
- added link slider_11_track, mass 0.1; collision box size=0.4479720179640173 0.005 0.02; visual box size=0.4479720179640173 0.005 0.02
Joints:
- removed joint slider_72_joint
- removed joint slider_72_track_joint
- added joint slider_11_joint: type prismatic, parent back_link, child slider_11_handle, origin xyz=-0.0654473394799941 0.05 0.034140619425656604 rpy=1.57 0 0, axis -0.4934206858851674 0.869790794812529 0, limit lower=-0.22398600898200866 upper=0.22398600898200866 effort=UNNAMED_10 velocity=UNNAMED_11
- added joint slider_11_track_joint: type fixed, parent back_link, child slider_11_track, origin xyz=-0.0654473394799941 0.025 0.034140619425656604 rpy=0 -2.0868144811120013 0

Commit message: Added continual training method

File: models/busybox0.urdf (robot description, URDF)
Before this commit: robot busybox, 4 links, 3 joints
Links:
- removed link slider_11_handle
- removed link slider_11_track
- added link slider_13_handle, mass 0.1; collision cylinder length=0.05 radius=0.02; visual cylinder length=0.05 radius=0.02
- added link slider_13_track, mass 0.1; collision box size=0.4959613416395672 0.005 0.02; visual box size=0.4959613416395672 0.005 0.02
Joints:
- removed joint slider_11_joint
- removed joint slider_11_track_joint
- added joint slider_13_joint: type prismatic, parent back_link, child slider_13_handle, origin xyz=-0.0318636095201309 0.05 -0.15412396644716406 rpy=1.57 0 0, axis -0.9488228370213238 0.31580884083066213 0, limit lower=-0.2479806708197836 upper=0.2479806708197836 effort=UNNAMED_10 velocity=UNNAMED_11
- added joint slider_13_track_joint: type fixed, parent back_link, child slider_13_track, origin xyz=-0.0318636095201309 0.025 -0.15412396644716406 rpy=0 -2.8202836526317685 0

Commit message: Modified evaluation

File: models/busybox0.urdf (robot description, URDF)
Before this commit: robot busybox, 4 links, 3 joints
Links:
- removed link slider_13_handle
- removed link slider_13_track
- added link slider_2_handle, mass 0.1; collision cylinder length=0.05 radius=0.02; visual cylinder length=0.05 radius=0.02
- added link slider_2_track, mass 0.1; collision box size=0.10743110160895926 0.005 0.02; visual box size=0.10743110160895926 0.005 0.02
Joints:
- removed joint slider_13_joint
- removed joint slider_13_track_joint
- added joint slider_2_joint: type prismatic, parent back_link, child slider_2_handle, origin xyz=0.011738085164543666 0.05 0.024457010836680226 rpy=1.57 0 0, axis -0.45640013771751753 0.8897746424187594 0, limit lower=-0.05371555080447963 upper=0.05371555080447963 effort=UNNAMED_3 velocity=UNNAMED_2
- added joint slider_2_track_joint: type fixed, parent back_link, child slider_2_track, origin xyz=0.011738085164543666 0.025 0.024457010836680226 rpy=0 -2.044741493916277 0
